File: reload.brd (EAGLE design)
At the start: 49.2 x 30.5 mm, 21 parts, among them IC1 MCP6002, IC2 LP2950Z, Q1 BTS117

Commit message: Board rearrangement for spring terminals, better pot placement.
Parts:
- JP1: device SparkFun-Connectors:SCREWTERMINAL-5MM-2 -> nickparts:SPRINGTERMINAL-5MM-2
- moved IC2 13.0 mm to (19.7, 26.4)
- moved C3 12.5 mm to (16.8, 21.3)
- moved C2 9.16 mm to (34.6, 27.0), turned to 180 degrees
- moved D1 8.89 mm to (19.4, 17.8)
- moved R3 7.63 mm to (26.7, 29.2)
- moved R6 5.41 mm to (26.7, 20.0)
- moved C1 5.17 mm to (38.7, 7.62), turned to 0 degrees
- moved R1 2.86 mm to (35.6, 15.2)
- moved JP1 1.59 mm to (44.1, 12.7)
Connections:
- removed net N$3: R3.P$1, R6.P$1
- new net N$2: R3.P$1, R6.P$3
- net GND: now also R6.P$1; no longer R6.P$3
Routing:
- net VCC: track 30.8 -> 55.8 mm
- net SENSE: track 74.5 -> 58.0 mm
- net N$8: track 6.90 -> 15.5 mm
- net N$3: track 7.36 -> 0.00 mm
- net V+: track 63.0 -> 58.0 mm
- net N$2: track 0.00 -> 2.75 mm
- net GND: track 89.7 -> 91.1 mm
- net N$7: track 8.92 -> 7.65 mm
- net N$4: track 17.8 -> 16.5 mm
