File: reload.brd (EAGLE design)
At the start: 50 x 31 mm, 22 parts, among them IC1 OPAMP-DUALMS, IC2 V_REG_MIC2920, Q1 BTS117

Commit message: Layout tweaks and updated images
Parts:
- added Q2: BTS117, SparkFun-DiscreteSemi:TO220V
- added SJ1: (no value), SparkFun-Passives:SJ_3_PASTE2&3
- added SJ2: (no value), SparkFun-Passives:SJ_3_PASTE1&2
- moved C3 1.27 mm to (16.5, 14.0)
- moved C5 1.27 mm to (20.3, 14.0)
- moved JP2 1.27 mm to (12.0, 14.8)
- moved IC2 0.95 mm to (18.7, 21.0)
Connections:
- new net N$10: R3.1, SJ1.3, SJ2.3
- new net N$8: R6.P$1, SJ2.2
- net GND: now also SJ1.1, SJ2.1; no longer R6.P$1
- net N$2: now also SJ1.2; no longer R3.1
- net N$3: now also Q2.3
- net N$9: now also Q2.1
- net V+: now also Q2.2
Routing:
- net N$8: track 0.00 -> 10.9 mm
- net N$10: track 0.00 -> 4.70 mm
- net N$3: track 42.8 -> 46.4 mm
- net N$9: track 10.7 -> 14.3 mm
- net V+: track 49.4 -> 51.8 mm
- net GND: track 86.9 -> 89.2 mm, vias 4 -> 5
- net N$2: track 13.1 -> 11.7 mm
- net VDD: track 43.1 -> 44.2 mm
- net VCC: track 14.5 -> 15.5 mm

Commit message: Tweaks and new Re:load images
Parts:
- Q2: device SparkFun-DiscreteSemi:TO220V -> nickparts:TO220V-NOSILK
- R2: device nickparts:TRIMPOT-3MM-2 -> nickparts:TRIMPOT-EVN5E
Changed lines of the file:
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@@
 </element>
 <element name="Q1" library="SparkFun-DiscreteSemi" package="TO220V" value="BTS117" x="6.6675" y="15.24" smashed="yes" rot="R90">
-<attribute name="NAME" x="2.921" y="15.3035" size="1.27" layer="25" ratio="10" rot="R90" align="bottom-center"/>
+<attribute name="NAME" x="6.2865" y="21.971" size="1.27" layer="25" ratio="10" rot="R180" align="bottom-center"/>
 </element>
 <element name="J1" library="SparkFun-Connectors" package="BANANA_CONN" value="" x="45.085" y="24.765"/>
@@
 </element>
 <element name="KK1" library="nickparts" package="SK129" value="SK129-PAD" x="1.5875" y="15.24" smashed="yes" rot="R90"/>
-<element name="R2" library="nickparts" package="TRIMPOT-3MM-2" value="1k" x="26.035" y="3.175" smashed="yes" rot="R270">
+<element name="R2" library="nickparts" package="TRIMPOT-EVN5E" value="1k" x="26.035" y="3.175" smashed="yes" rot="R270">
 <attribute name="NAME" x="25.5905" y="3.302" size="0.8128" layer="25" rot="R270" align="bottom-center"/>
 </element>
@@
 <attribute name="VALUE" x="22.352" y="13.843" size="0.4064" layer="27"/>
 </element>
-<element name="Q2" library="SparkFun-DiscreteSemi" package="TO220V" value="BTS117" x="3.048" y="15.24" rot="R90"/>
+<element name="Q2" library="nickparts" package="TO220V-NOSILK" value="BTS117" x="3.048" y="15.24" rot="R90"/>
 </elements>
 <signals>
@@
 <contactref element="R4" pad="2"/>
 <contactref element="R2" pad="3"/>
-<wire x1="24.235" y1="2.175" x2="24.665" y2="2.33375" width="0.254" layer="1"/>
-<wire x1="24.3225" y1="2.2225" x2="24.235" y2="2.175" width="0.254" layer="1"/>
+<wire x1="24.435" y1="2.175" x2="24.665" y2="2.33375" width="0.254" layer="1"/>
+<wire x1="24.3225" y1="2.2225" x2="24.435" y2="2.175" width="0.254" layer="1"/>
 <wire x1="22.49" y1="1.905" x2="23.965" y2="1.905" width="0.254" layer="1"/>
-<wire x1="23.965" y1="1.905" x2="24.235" y2="2.175" width="0.254" layer="1"/>
+<wire x1="23.965" y1="1.905" x2="24.435" y2="2.175" width="0.254" layer="1"/>
 </signal>
 <signal name="N$5">
 <contactref element="R2" pad="2"/>
 <contactref element="IC1" pad="6"/>
-<wire x1="27.73125" y1="3.175" x2="27.485" y2="3.175" width="0.1524" layer="1"/>
+<wire x1="27.73125" y1="3.175" x2="27.535" y2="3.175" width="0.1524" layer="1"/>
 <wire x1="31.75" y1="14.03" x2="31.75" y2="15.24" width="0.1524" layer="1"/>
 <wire x1="31.75" y1="15.24" x2="32.0675" y2="15.5575" width="0.1524" layer="1"/>
@@
 <wire x1="35.925" y1="6.3975" x2="33.3375" y2="3.81" width="0.1524" layer="1"/>
 <wire x1="33.3375" y1="3.81" x2="28.12" y2="3.81" width="0.1524" layer="1"/>
-<wire x1="28.12" y1="3.81" x2="27.485" y2="3.175" width="0.1524" layer="1"/>
+<wire x1="28.12" y1="3.81" x2="27.535" y2="3.175" width="0.1524" layer="1"/>
 </signal>
 <signal name="N$6">
 <contactref element="R5" pad="1"/>
 <contactref element="R2" pad="1"/>
-<wire x1="24.235" y1="4.175" x2="24.665" y2="4.33375" width="0.254" layer="1"/>
+<wire x1="24.435" y1="4.175" x2="24.665" y2="4.33375" width="0.254" layer="1"/>
 <wire x1="22.49" y1="4.445" x2="23.965" y2="4.445" width="0.254" layer="1"/>
-<wire x1="23.965" y1="4.445" x2="24.235" y2="4.175" width="0.254" layer="1"/>
+<wire x1="23.965" y1="4.445" x2="24.435" y2="4.175" width="0.254" layer="1"/>
 </signal>
 <signal name="N$1">

Commit message: Added complete technical BoM and updated schematic as so politely suggested by a commenter
Parts:
- IC1: value OPAMP-DUALMS -> MCP6002
- IC2: value V_REG_MIC2920 -> LM2936-3.0
Changed lines of the file:
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@@
 <element name="U$2" library="nickparts" package="ARACHNID_LABS_LOGO_SM" value="" x="20.75" y="15.24" rot="MR270"/>
 <element name="U$3" library="SparkFun-Aesthetics" package="OSHW-LOGO-M" value="" x="11.86" y="15.24" rot="MR270"/>
-<element name="IC1" library="nickparts" package="SOP08" value="OPAMP-DUALMS" x="31.115" y="11.43" smashed="yes">
+<element name="IC1" library="nickparts" package="SOP08" value="MCP6002" x="31.115" y="11.43" smashed="yes">
 <attribute name="NAME" x="31.115" y="11.43" size="0.8128" layer="25" align="bottom-center"/>
 </element>
-<element name="IC2" library="SparkFun-PowerIC" package="SOT223" value="V_REG_MIC2920" x="18.7325" y="20.955" smashed="yes">
+<element name="IC2" library="SparkFun-PowerIC" package="SOT223" value="LM2936-3.0" x="18.7325" y="20.955" smashed="yes">
 <attribute name="NAME" x="18.7325" y="20.955" size="0.8128" layer="25" align="bottom-center"/>
 </element>
@@
 </signal>
 </signals>
-<errors>
-</errors>
 </board>
 </drawing>
