File: reload.sch (EAGLE design)
At the start: 20 parts, among them IC1 OPAMP-DUALMS, IC2 V_REG_MIC2920, Q1 BTS117

Commit message: Layout tweaks and updated images
Parts:
- added Q2: BTS117, SparkFun-DiscreteSemi:MOSFET-NCHANNELPTH2
- added SJ1: (no value), SparkFun-Passives:SOLDERJUMPER_2WAYPASTE2&3
- added SJ2: (no value), SparkFun-Passives:SOLDERJUMPER_2WAYPASTE1&2
Connections:
- new net N$10: R3.1, SJ1.3, SJ2.3
- new net N$8: R6.E, SJ2.2
- net GND: now also SJ1.1, SJ2.1; no longer R6.E
- net N$2: now also SJ1.2; no longer R3.1
- net N$3: now also Q2.S
- net N$9: now also Q2.G
- net V+: now also Q2.D
Other:
- moved on the sheet: R3
Changed lines of the file:
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@@
 <part name="SUPPLY2" library="supply2" deviceset="VDD" device=""/>
 <part name="C5" library="SparkFun-Passives" deviceset="CAP" device="0805" value="22u"/>
+<part name="SJ1" library="SparkFun-Passives" deviceset="SOLDERJUMPER_2WAY" device="PASTE2&amp;3"/>
+<part name="SJ2" library="SparkFun-Passives" deviceset="SOLDERJUMPER_2WAY" device="PASTE1&amp;2"/>
+<part name="GND8" library="supply1" deviceset="GND" device=""/>
+<part name="Q2" library="SparkFun-DiscreteSemi" deviceset="MOSFET-NCHANNEL" device="PTH2" value="BTS117"/>
+<part name="P+6" library="supply1" deviceset="V+" device=""/>
 </parts>
 <sheets>
@@
 <instance part="GND2" gate="1" x="111.76" y="93.98"/>
 <instance part="R6" gate="G$1" x="96.52" y="101.6" rot="MR180"/>
-<instance part="GND3" gate="1" x="96.52" y="91.44"/>
-<instance part="R3" gate="G$1" x="96.52" y="114.3" rot="R90"/>
+<instance part="GND3" gate="1" x="91.44" y="81.28"/>
+<instance part="R3" gate="G$1" x="96.52" y="119.38" rot="R90"/>
 <instance part="GND4" gate="1" x="48.26" y="25.4"/>
 <instance part="P+3" gate="1" x="15.24" y="58.42"/>
@@
 <instance part="R7" gate="G$1" x="132.08" y="104.14" rot="R180"/>
 <instance part="P+2" gate="VCC" x="60.96" y="58.42"/>
-<instance part="P+5" gate="VCC" x="96.52" y="121.92"/>
+<instance part="P+5" gate="VCC" x="96.52" y="127"/>
 <instance part="RELOAD" gate="G$1" x="0" y="0"/>
 <instance part="RELOAD" gate="G$2" x="147.32" y="0"/>
@@
 <instance part="SUPPLY2" gate="G$1" x="226.06" y="119.38"/>
 <instance part="C5" gate="G$1" x="60.96" y="43.18"/>
+<instance part="SJ1" gate="G$1" x="91.44" y="109.22" rot="R180"/>
+<instance part="SJ2" gate="G$1" x="91.44" y="88.9" rot="R180"/>
+<instance part="GND8" gate="1" x="91.44" y="101.6"/>
+<instance part="Q2" gate="G$1" x="157.48" y="96.52"/>
+<instance part="P+6" gate="1" x="157.48" y="104.14"/>
 </instances>
 <busses>
@@
 <pinref part="P+3" gate="1" pin="V+"/>
 <wire x1="15.24" y1="55.88" x2="22.86" y2="55.88" width="0.1524" layer="91"/>
+</segment>
+<segment>
+<pinref part="Q2" gate="G$1" pin="D"/>
+<pinref part="P+6" gate="1" pin="V+"/>
 </segment>
 </net>
@@
 </segment>
 <segment>
-<pinref part="GND3" gate="1" pin="GND"/>
-<pinref part="R6" gate="G$1" pin="E"/>
-</segment>
-<segment>
 <pinref part="JP1" gate="G$1" pin="1"/>
 <pinref part="GND6" gate="1" pin="GND"/>
 <wire x1="228.6" y1="109.22" x2="226.06" y2="109.22" width="0.1524" layer="91"/>
 <wire x1="226.06" y1="109.22" x2="226.06" y2="106.68" width="0.1524" layer="91"/>
+</segment>
+<segment>
+<pinref part="SJ2" gate="G$1" pin="1"/>
+<pinref part="GND3" gate="1" pin="GND"/>
+</segment>
+<segment>
+<pinref part="SJ1" gate="G$1" pin="1"/>
+<pinref part="GND8" gate="1" pin="GND"/>
 </segment>
 </net>
@@
 <pinref part="Q1" gate="G$1" pin="G"/>
 <wire x1="137.16" y1="104.14" x2="139.7" y2="104.14" width="0.1524" layer="91"/>
+<pinref part="Q2" gate="G$1" pin="G"/>
+<wire x1="149.86" y1="96.52" x2="139.7" y2="96.52" width="0.1524" layer="91"/>
+<wire x1="139.7" y1="96.52" x2="139.7" y2="104.14" width="0.1524" layer="91"/>
+<junction x="139.7" y="104.14"/>
 </segment>
 </net>
@@
 <wire x1="111.76" y1="114.3" x2="111.76" y2="111.76" width="0.1524" layer="91"/>
 <wire x1="124.46" y1="114.3" x2="111.76" y2="114.3" width="0.1524" layer="91"/>
-<wire x1="96.52" y1="119.38" x2="111.76" y2="119.38" width="0.1524" layer="91"/>
-<wire x1="111.76" y1="119.38" x2="111.76" y2="114.3" width="0.1524" layer="91"/>
-<junction x="96.52" y="119.38"/>
+<wire x1="96.52" y1="124.46" x2="111.76" y2="124.46" width="0.1524" layer="91"/>
+<wire x1="111.76" y1="124.46" x2="111.76" y2="114.3" width="0.1524" layer="91"/>
+<junction x="96.52" y="124.46"/>
 <junction x="111.76" y="114.3"/>
 <pinref part="P+5" gate="VCC" pin="VCC"/>
 <pinref part="IC1" gate="A" pin="V+"/>
-</segment>
-</net>
-<net name="N$2" class="0">
-<segment>
-<pinref part="R3" gate="G$1" pin="1"/>
-<pinref part="R6" gate="G$1" pin="A"/>
 </segment>
 </net>
@@
 <wire x1="147.32" y1="88.9" x2="147.32" y2="99.06" width="0.1524" layer="91"/>
 <junction x="147.32" y="88.9"/>
+<pinref part="Q2" gate="G$1" pin="S"/>
+<wire x1="157.48" y1="91.44" x2="157.48" y2="88.9" width="0.1524" layer="91"/>
+<wire x1="157.48" y1="88.9" x2="147.32" y2="88.9" width="0.1524" layer="91"/>
 </segment>
 </net>
@@
 </segment>
 </net>
+<net name="N$2" class="0">
+<segment>
+<pinref part="R6" gate="G$1" pin="A"/>
+<pinref part="SJ1" gate="G$1" pin="2"/>
+</segment>
+</net>
+<net name="N$8" class="0">
+<segment>
+<pinref part="R6" gate="G$1" pin="E"/>
+<pinref part="SJ2" gate="G$1" pin="2"/>
+<wire x1="96.52" y1="88.9" x2="96.52" y2="93.98" width="0.1524" layer="91"/>
+</segment>
+</net>
+<net name="N$10" class="0">
+<segment>
+<pinref part="R3" gate="G$1" pin="1"/>
+<pinref part="SJ1" gate="G$1" pin="3"/>
+<wire x1="96.52" y1="114.3" x2="91.44" y2="114.3" width="0.1524" layer="91"/>
+<pinref part="SJ2" gate="G$1" pin="3"/>
+<wire x1="91.44" y1="93.98" x2="83.82" y2="93.98" width="0.1524" layer="91"/>
+<wire x1="83.82" y1="93.98" x2="83.82" y2="114.3" width="0.1524" layer="91"/>
+<wire x1="83.82" y1="114.3" x2="91.44" y2="114.3" width="0.1524" layer="91"/>
+<junction x="91.44" y="114.3"/>
+</segment>
+</net>

Commit message: Tweaks and new Re:load images
Parts:
- Q2: device SparkFun-DiscreteSemi:MOSFET-NCHANNELPTH2 -> nickparts:MOSFET-NCHANNELTO220V-NOSILK
- R2: device nickparts:TRIMPOT3MM-2 -> nickparts:TRIMPOTEVN5E
Changed lines of the file:
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@@
 <part name="C3" library="SparkFun-Passives" deviceset="CAP" device="0805" value="1u"/>
 <part name="KK1" library="nickparts" deviceset="SK129-PAD" device=""/>
-<part name="R2" library="nickparts" deviceset="TRIMPOT" device="3MM-2" value="1k"/>
+<part name="R2" library="nickparts" deviceset="TRIMPOT" device="EVN5E" value="1k"/>
 <part name="R7" library="SparkFun-Passives" deviceset="RESISTOR" device="0805-RES" value="100"/>
 <part name="P+2" library="supply1" deviceset="VCC" device=""/>
@@
 <part name="SJ2" library="SparkFun-Passives" deviceset="SOLDERJUMPER_2WAY" device="PASTE1&amp;2"/>
 <part name="GND8" library="supply1" deviceset="GND" device=""/>
-<part name="Q2" library="SparkFun-DiscreteSemi" deviceset="MOSFET-NCHANNEL" device="PTH2" value="BTS117"/>
+<part name="Q2" library="nickparts" deviceset="MOSFET-NCHANNEL" device="TO220V-NOSILK" value="BTS117"/>
 <part name="P+6" library="supply1" deviceset="V+" device=""/>
 </parts>

Commit message: Added complete technical BoM and updated schematic as so politely suggested by a commenter
Parts:
- IC1: value OPAMP-DUALMS -> MCP6002
- IC2: value V_REG_MIC2920 -> LM2936-3.0
Other:
- note added: "Two footprints for Q1 Populate only one"
Changed lines of the file:
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@@
 <part name="P+5" library="supply1" deviceset="VCC" device=""/>
 <part name="RELOAD" library="SparkFun-Aesthetics" deviceset="FRAME-LETTER" device=""/>
-<part name="IC1" library="nickparts" deviceset="OPAMP-DUAL" device="MS"/>
-<part name="IC2" library="SparkFun-PowerIC" deviceset="V_REG_MIC2920" device=""/>
+<part name="IC1" library="nickparts" deviceset="OPAMP-DUAL" device="MS" value="MCP6002"/>
+<part name="IC2" library="SparkFun-PowerIC" deviceset="V_REG_MIC2920" device="" value="LM2936-3.0"/>
 <part name="JP1" library="SparkFun-Connectors" deviceset="M03" device="1X03_NO_SILK"/>
 <part name="R8" library="SparkFun-Passives" deviceset="RESISTOR" device="0805-RES" value="10k 1%"/>
@@
 <text x="210.82" y="180.34" size="3.81" layer="94" align="bottom-center">Current Reading</text>
 <text x="200.66" y="7.62" size="2.54" layer="94" align="bottom-center">Arachnid Labs (Nick Johnson)</text>
+<text x="152.4" y="114.3" size="1.778" layer="97" align="bottom-center">Two footprints for Q1
+Populate only one</text>
 </plain>
 <instances>
@@
 </schematic>
 </drawing>
+<compatibility>
+<note version="6.3" minversion="6.2.2" severity="warning">
+Since Version 6.2.2 text objects can contain more than one line,
+which will not be processed correctly with this version.
+</note>
+</compatibility>
 </eagle>
